Commit message: updated the aprilTag version

File: fruitSorter/urdf/green_cube.urdf (robot description, URDF)
Before this commit: robot green_cube, 1 links, 0 joints
Links:
- link base_link: mass 0.1 -> 0.0225; geometry collision box size=0.0318 0.0318 0.0318; visual box size=0.0318 0.0318 0.0318

File: fruitSorter/urdf/red_cube.urdf (robot description, URDF)
Before this commit: robot red_cube, 1 links, 0 joints
Links:
- link base_link: mass 0.1 -> 0.0225; geometry collision box size=0.0318 0.0318 0.0318; visual box size=0.0318 0.0318 0.0318
